Commit message: Added .stl and some stuffs.

File: model/calibrator.urdf.xacro (robot description, xacro)
@@ -1,32 +1,36 @@
 <?xml version="1.0"?>
 <robot xmlns:xacro="http://www.ros.org/wiki/xacro">
-<xacro:macro name="calibrator" params="parent name *origin">
-  <joint name="${parent}_${name}_base_joint" type="fixed">
-    <xacro:insert_block name="origin"/>
-    <parent link="${parent}"/>
-    <child link="${name}_mesh"/>
-  </joint>
-  <link name="${name}_mesh">
-    <visual>
-      <geometry>
-        <mesh filename="package://calibration/meshes/camera_robot_calibrator.stl"/>
-      </geometry>
-      <material name="Vito/Silver"/>
-    </visual>
-    <collision>
-      <geometry>
-        <mesh filename="package://calibration/meshes/camera_robot_calibrator.stl"/>
-      </geometry>
-    </collision>
-  </link>
-  <!-- this is where the ar marker is w.r.t. the mesh, known from CAD model -->
-  <joint name="${name}_joint" type="fixed">
-    <origin xyz="0 0 0.02" rpy="   1.570796326794897 0 0"/>
-    <!-- <origin xyz="0 0 0.02" rpy="0 0 0"/> -->
-<!--  -->
-  <parent link="${name}_mesh"/>
-    <child link="${name}"/>
-  </joint>
-  <link name="${name}"/>
-</xacro:macro>
+  <xacro:macro name="calibrator" params="parent name *origin">
+    <joint name="${parent}_${name}_base_joint" type="fixed">
+      <xacro:insert_block name="origin" />
+      <parent link="${parent}" />
+      <child link="${name}_mesh" />
+    </joint>
+    <link name="${name}_mesh">
+      <visual>
+        <origin xyz="0 0 0" rpy="1.57 0 0"/>
+        <geometry>
+          <mesh filename="package://calibration/meshes/camera_robot_calibrator.stl" />
+        </geometry>
+        <!-- <material name="Vito/Silver" /> -->
+        <material name="Cyan">
+                 <color rgba="0 1.0 1.0 1.0"/>
+        </material>
+      </visual>
+      <collision>
+        <geometry>
+          <mesh filename="package://calibration/meshes/camera_robot_calibrator.stl" />
+        </geometry>
+      </collision>
+    </link>
+    <!-- this is where the ar marker is w.r.t. the mesh, known from CAD model -->
+    <joint name="${name}_joint" type="fixed">
+      <origin xyz="0 -0.02 0" rpy="1.570796326794897 0 0" />
+      <!-- <origin xyz="0 0 0.02" rpy="0 0 0"/> -->
+      <!--  -->
+      <parent link="${name}_mesh" />
+      <child link="${name}" />
+    </joint>
+    <link name="${name}" />
+  </xacro:macro>
 </robot>

File: robots/panda_arm_calibration.urdf.xacro (robot description, xacro)
@@ -1,6 +1,6 @@
 <?xml version='1.0' encoding='utf-8'?>
 <robot xmlns:xacro="http://www.ros.org/wiki/xacro" name="panda">
-  <xacro:include filename="$(find franka_description)/robots/common/franka_robot.xacro"/>
-      <xacro:include filename="$(find calibration)/model/calibrator.urdf.xacro"/>
+  <xacro:include filename="$(find franka_description)/robots/common/franka_robot.xacro" />
+  <xacro:include filename="$(find calibration)/model/calibrator.urdf.xacro" />
   <xacro:arg name="arm_id" default="panda" />
   <!-- Should a franka_gripper be mounted at the flange?" -->
@@ -8,27 +8,25 @@
   <!-- Positional offset between $(arm_id)_hand -> $(arm_id)_hand_tcp [m]. Only used when hand:=true -->
   <xacro:arg name="tcp_xyz" default="0 0 0.1034" />
-  <!-- Rotational offset between $(arm_id)_hand -> $(arm_id)_hand_tcp [rad]. Only used when hand:=true -->
+  <!-- Rotational offset between $(arm_id)_hand -> $(arm_id)_hand_tcp [rad]. Only used when
+  hand:=true -->
   <xacro:arg name="tcp_rpy" default="0 0 0" />
   <!-- Is the robot being simulated in gazebo?" -->
   <xacro:arg name="gazebo" default="false" />
-  <!-- If `gazebo` arg is set, to which frame shall $(arm_id)_link0 be parented. Empty string for not fixing at all -->
+  <!-- If `gazebo` arg is set, to which frame shall $(arm_id)_link0 be parented. Empty string for
+  not fixing at all -->
   <xacro:arg name="parent" default="world" />
-  <!-- If `gazebo` arg is set and `parent` not empty, what position offset between `parent` & $(arm_id)_link0 -->
+  <!-- If `gazebo` arg is set and `parent` not empty, what position offset between `parent` &
+  $(arm_id)_link0 -->
   <xacro:arg name="xyz" default="0 0 0" />
-  <!-- If `gazebo` arg is set and `parent` not empty, what rotation offset between `parent` & $(arm_id)_link0 -->
+  <!-- If `gazebo` arg is set and `parent` not empty, what rotation offset between `parent` &
+  $(arm_id)_link0 -->
   <xacro:arg name="rpy" default="0 0 0" />
   <xacro:franka_robot arm_id="$(arg arm_id)"
-                      joint_limits="${xacro.load_yaml('$(find franka_description)/robots/panda/joint_limits.yaml')}"
-                      hand="$(arg hand)"
-                      tcp_xyz="$(arg tcp_xyz)"
-                      tcp_rpy="$(arg tcp_rpy)"
-                      gazebo="$(arg gazebo)"
-                      parent="$(arg parent)"
-                      xyz="$(arg xyz)"
-                      rpy="$(arg rpy)">
+    joint_limits="${xacro.load_yaml('$(find franka_description)/robots/panda/joint_limits.yaml')}"
+  >
   </xacro:franka_robot>
   <!-- from the CAD model, the frame coincides with the 7-th link -->
   <xacro:calibrator name="calibrator_10" parent="panda_link8">
-    <origin xyz="0 0 0" rpy="0 0 0"/>
+    <origin xyz="0 0 0" rpy="-1.57 0 0" />
   </xacro:calibrator>
 </robot>
